File: controlcarreta.kicad_sch (KiCad schematic)
At the start: 92 parts, among them J1 Screw_Terminal_01x02, J10 MOLEX10POS, J11 MOLEX10POS, J1255 Conn_Coaxial, J13 USB-C 2.0, J14 Mini PCIe Socket 52p, J15 nano-SIM, J16 u.FL, J17 RS-232 DE9 (M,DTE), J2 Screw_Terminal_01x02, J3 Conn_01x04_Male, J4 MOLEX10POS, J5 MOLEX10POS, J6 MOLEX10POS, J7 MOLEX10POS, J8 MOLEX10POS, J9 MOLEX10POS, Q1 SI4447ADY-T1-GE3, SW1 RESET, SW2 BOOT, U1 ESP32-S3-WROOM-1-N8, U10 LM2596S-ADJ, U11 MAX3232E, U2 LM2596S-ADJ, U3 sdcard, U4 74LVC8T245PW-Q100J, U5 74LVC8T245PW-Q100J, U6 74LVC8T245PW-Q100J, U8 NCP1117-3.3, U9 USBLC6-2SC6

Commit message: home parcial ordered
Parts:
- removed C1, C3: 100 uF, Capacitor_SMD:CP_Elec_8x10.5, symbol Device:CP
- removed C10, C12: 10uF, Capacitor_SMD:C_0805_2012Metric_Pad1.18x1.45mm_HandSolder, symbol Device:C
- removed C11: 22uF, Capacitor_SMD:C_0805_2012Metric_Pad1.18x1.45mm_HandSolder, symbol Device:C
- removed C13, C22, C27, C28, C29, C30, C31, C32: 100nF, Capacitor_SMD:C_0805_2012Metric_Pad1.18x1.45mm_HandSolder, symbol Device:C
- removed C2: 1500 pF, Capacitor_SMD:C_0805_2012Metric_Pad1.18x1.45mm_HandSolder, symbol pspice:CAP
- removed C24: 1.5nF, Capacitor_SMD:C_0805_2012Metric_Pad1.18x1.45mm_HandSolder, symbol Device:C
- removed C25: 100uF, Capacitor_SMD:CP_Elec_8x10.5, symbol Device:C
- removed C26: 470uF, Capacitor_SMD:CP_Elec_10x10.5, symbol Device:C
- removed C4, C6, C7, C8: 4.7 uF, Capacitor_SMD:C_0805_2012Metric_Pad1.18x1.45mm_HandSolder, symbol pspice:C
- removed D1: D_Zener, Diode_SMD:D_2114_3652Metric, symbol Device:D_Zener
- removed D7: SS14, Diode_SMD:D_SMA, symbol Device:D_Schottky
- removed D8: SS34, Diode_SMD:D_SMA, symbol Device:D_Schottky
- removed D9: WWAN, LED_SMD:LED_0805_2012Metric, symbol Device:LED
- removed J10, J11, J4, J5, J6, J7, J8, J9: MOLEX10POS, MOLEX10POS:MOLEX10POS, symbol MOLEX10POS:MOLEX10POS
- removed J13: USB-C 2.0, Connector_USB:USB_C_Receptacle_GCT_USB4085, symbol Connector:USB_C_Receptacle_USB2.0_16P
- removed J14: Mini PCIe Socket 52p, Connector_PCBEdge:BUS_PCI_Express_Mini_Full, symbol Connector:Bus_PCI_Express_Mini
- removed J15: nano-SIM, Connector_Card:nanoSIM_Hinged_CUI_NSIM-2-C, symbol Connector:SIM_Card
- removed J16: u.FL, Connector_Coaxial:U.FL_Hirose_U.FL-R-SMT-1_Vertical, symbol Connector:Conn_Coaxial
- removed J17: RS-232 DE9 (M,DTE), Connector_Dsub:DSUB-9_Pins_Horizontal_P2.77x2.84mm_EdgePinOffset9.40mm, symbol Connector:DE9_Pins
- removed L1: INDUCTOR, Inductor_SMD:L_Bourns_SDR1806, symbol pspice:INDUCTOR
- removed L2: 33uH, Inductor_SMD:L_Bourns_SDR1806, symbol pspice:INDUCTOR
- removed R1, R24, R26: 1k, Resistor_SMD:R_1206_3216Metric_Pad1.30x1.75mm_HandSolder, symbol Device:R
- removed R15, R16: 5.1k, Resistor_SMD:R_1206_3216Metric_Pad1.30x1.75mm_HandSolder, symbol Device:R
- removed R2: 3k, Resistor_SMD:R_1206_3216Metric_Pad1.30x1.75mm_HandSolder, symbol Device:R
- removed R20, R21: 10k, Resistor_SMD:R_1206_3216Metric_Pad1.30x1.75mm_HandSolder, symbol Device:R
- removed R25: 1.69k, Resistor_SMD:R_1206_3216Metric_Pad1.30x1.75mm_HandSolder, symbol Device:R
- removed R27: 0R, Resistor_SMD:R_1206_3216Metric_Pad1.30x1.75mm_HandSolder, symbol Device:R
- removed U10, U2: LM2596S-ADJ, Package_TO_SOT_SMD:TO-263-5_TabPin3, symbol Regulator_Switching:LM2596S-ADJ
- removed U11: MAX3232E, Package_SO:SOIC-16_3.9x9.9mm_P1.27mm, symbol controlcarreta:MAX3232
- removed U3: sdcard, sdcard:sdcardgoia, symbol sdcard:sdcard
- removed U4, U5, U6: 74LVC8T245PW-Q100J, Package_SO:TSSOP-24_4.4x7.8mm_P0.65mm, symbol 74LVC8T245PW:74LVC8T245PW
- removed U8: NCP1117-3.3, Package_TO_SOT_SMD:SOT-223-3_TabPin2, symbol controlcarreta:NCP1117-3.3_SOT223
- removed U9: USBLC6-2SC6, Package_TO_SOT_SMD:SOT-23-6, symbol controlcarreta:USBLC6-2SC6
Connections:
- no-connect marks 91 -> 3
Other:
- added sheet DRIVERS (drivers.kicad_sch)
- added sheet LDO_3V3 (ldo_3v3.kicad_sch)
- added sheet MODEM (modem.kicad_sch)
- added sheet PSU_5V (psu_5v.kicad_sch)
- added sheet PSU_MODEM (psu_modem.kicad_sch)
- added sheet RS232 (rs232.kicad_sch)
- added sheet SDCARD (sdcard.kicad_sch)
- added sheet USB (usb.kicad_sch)

Commit message: WIP: J18/Q2/Q3/R30/R31 + reguardado KiCad de todas las hojas
Parts:
- added J18: FTDI_AUTOPROG, Connector_PinHeader_2.54mm:PinHeader_1x06_P2.54mm_Vertical, symbol Connector:Conn_01x06_Pin
- added Q2, Q3: SS8050, Package_TO_SOT_SMD:SOT-23, symbol Transistor_BJT:Q_NPN_BEC
- added R30, R31: 12k, Resistor_SMD:R_1206_3216Metric_Pad1.30x1.75mm_HandSolder, symbol Device:R
Connections:
- net +3.3V: now also J18.4 (Pin_4)
- net EN: now also Q2.3 (C)
- net GND: now also J18.6 (Pin_6)
- net IO0: now also Q3.3 (C)
- net RX_EXT: now also J18.3 (Pin_3)
- net TX_EXT: now also J18.2 (Pin_2)
- new net: Q2.2 (E), Q3.1 (B), R31.2
- new net: Q2.1 (B), Q3.2 (E), R30.2
- new net DTR: J18.1 (Pin_1), R30.1
- new net RTS: J18.5 (Pin_5), R31.1
Other:
- note added: "AUTO-PROGRAM: FT232 DTR/RTS -> EN/IO0 (esptool default_reset)"
