File: controlcarreta.kicad_sch (KiCad schematic)
At the start: 38 parts, among them J1 Screw_Terminal_01x02, J1255 Conn_Coaxial, J18 FTDI_AUTOPROG, J2 Screw_Terminal_01x02, J3 Conn_01x04_Male, Q1 SI4447ADY-T1-GE3, Q2 SS8050, Q3 SS8050, SW1 RESET, SW2 BOOT, U1 ESP32-S3-WROOM-1-N8

Commit message: modem: DTR (J14 pin 31) fuera de GND -> GPIO IO3 (net MODEM_DTR)
El EG25-G/SIM7600 no puede entrar en sleep con DTR a masa (idle ~20 mA
en vez de ~4 mA). Se suelta el pin 31 de GND y se lleva a U1 IO3
(GPIO libre, antes NO_CONNECT) via nueva senal jerarquica MODEM_DTR:
 - modem.kicad_sch: #PWR0551 (GND) -> hierarchical_label MODEM_DTR
 - controlcarreta.kicad_sch: pin de hoja MODEM_DTR + label en U1.15 (IO3),
   se elimina el no_connect de IO3

ERC sin cambios (370 warnings, 0 errores). Panel LED 7 se conserva:
habia 3 GPIO libres (IO3/IO45/IO46), no hacia falta sacrificarlo.

Co-Authored-By: Claude Sonnet 5 <noreply@anthropic.com>
Claude-Session: https://claude.ai/code/session_01T7LXaJdHR17hwkEUJr3uCL
Connections:
- net MODEM_DTR: now reaches U1.15 (IO3)
- no-connect marks 3 -> 2
Other:
- sheet MODEM ports: added MODEM_DTR; removed none
Changed lines of the file:
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@@
 		(color 0 0 0 0)
 	)
-	(no_connect
-		(at 44.45 111.76)
+	(wire
+		(pts
+			(xy 44.45 111.76) (xy 38.1 111.76)
+		)
+		(stroke
+			(width 0)
+			(type default)
+		)
+	)
+	(label "MODEM_DTR"
+		(at 38.1 111.76 180)
+		(effects
+			(font
+				(size 1.27 1.27)
+			)
+			(justify right bottom)
+		)
 	)
 	(no_connect
@@
 	(wire
 		(pts
+			(xy 330.2 106.68) (xy 320.04 106.68)
+		)
+		(stroke
+			(width 0)
+			(type default)
+		)
+	)
+	(label "MODEM_DTR"
+		(at 320.04 106.68 0)
+		(effects
+			(font
+				(size 1.27 1.27)
+			)
+			(justify right bottom)
+		)
+	)
+	(wire
+		(pts
 			(xy 201.295 182.245) (xy 201.295 183.515)
 		)
@@
 			(effects
 				(font
+					(size 1.27 1.27)
+				)
+				(justify right)
+			)
+		)
+		(pin "MODEM_DTR" bidirectional
+			(at 330.2 106.68 180)
+			(effects
+				(font
