File: modem.kicad_sch (KiCad schematic)
At the start: 9 parts, among them J14 Mini PCIe Socket 52p, J15 nano-SIM, J16 u.FL

Commit message: modem: DTR (J14 pin 31) fuera de GND -> GPIO IO3 (net MODEM_DTR)
El EG25-G/SIM7600 no puede entrar en sleep con DTR a masa (idle ~20 mA
en vez de ~4 mA). Se suelta el pin 31 de GND y se lleva a U1 IO3
(GPIO libre, antes NO_CONNECT) via nueva senal jerarquica MODEM_DTR:
 - modem.kicad_sch: #PWR0551 (GND) -> hierarchical_label MODEM_DTR
 - controlcarreta.kicad_sch: pin de hoja MODEM_DTR + label en U1.15 (IO3),
   se elimina el no_connect de IO3

ERC sin cambios (370 warnings, 0 errores). Panel LED 7 se conserva:
habia 3 GPIO libres (IO3/IO45/IO46), no hacia falta sacrificarlo.

Co-Authored-By: Claude Sonnet 5 <noreply@anthropic.com>
Claude-Session: https://claude.ai/code/session_01T7LXaJdHR17hwkEUJr3uCL
Connections:
- net GND: no longer J14.31 (PETn0)
- new net MODEM_DTR: J14.31 (PETn0)
Changed lines of the file:
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@@
 		)
 	)
-	(symbol
-		(lib_id "power:GND")
-		(at 175.26 101.6 0)
-		(unit 1)
-		(exclude_from_sim no)
-		(in_bom yes)
-		(on_board yes)
-		(dnp no)
-		(property "Reference" "#PWR0551"
-			(at 175.26 96.6 0)
-			(effects
-				(font
-					(size 1.27 1.27)
-				)
-				(justify left bottom)
-				(hide yes)
+	(hierarchical_label "MODEM_DTR"
+		(shape bidirectional)
+		(at 175.26 101.6 180)
+		(effects
+			(font
+				(size 1.27 1.27)
 			)
-		)
-		(property "Value" "GND"
-			(at 175.26 106.6 0)
-			(effects
-				(font
-					(size 1.27 1.27)
-				)
-				(justify left bottom)
-			)
-		)
-		(property "Footprint" ""
-			(at 175.26 101.6 0)
-			(effects
-				(font
-					(size 1.27 1.27)
-				)
-				(justify left bottom)
-				(hide yes)
-			)
-		)
-		(property "Datasheet" "~"
-			(at 175.26 101.6 0)
-			(effects
-				(font
-					(size 1.27 1.27)
-				)
-				(justify left bottom)
-				(hide yes)
-			)
-		)
-		(property "Description" ""
-			(at 175.26 101.6 0)
-			(effects
-				(font
-					(size 1.27 1.27)
-				)
-				(justify left bottom)
-				(hide yes)
-			)
-		)
-		(pin "1"
-		)
-		(instances
-			(project "controlcarreta"
-				(path "/9232987b-e923-413e-abd9-77ced6cc4c47/46e5d0ef-dab9-446e-ac53-867ecc660a13"
-					(reference "#PWR0551")
-					(unit 1)
-				)
-			)
+			(justify right)
 		)
 	)

Commit message: modem: 2a via de antena ANT_GNSS (J19 u.FL + J20 SMA) para GPS
El EG25-G / SIM7600 llevan receptor GNSS integrado pero necesitan
antena propia; el esquematico solo tenia ANT_MAIN. Se anade una 2a via
RF identica en topologia a ANT_MAIN:
 - modem.kicad_sch: J19 (u.FL Hirose) -> hierarchical_label ANT_GNSS,
   blindaje a GND (#PWR0563). Pigtail u.FL-u.FL a la toma GNSS de la
   tarjeta Mini-PCIe.
 - controlcarreta.kicad_sch: pin de hoja ANT_GNSS + J20 (SMA Amphenol)
   en la net ANT_GNSS, blindaje a GND (#PWR0564). Caja de la hoja MODEM
   ampliada (12.7 -> 17.78 mm) para alojar los 2 pines nuevos.
 - Poblar J19 O J20 (no ambos). Antena GNSS pasiva, vista al cielo,
   >=3 cm de ANT_MAIN.

ERC sin cambios (370 warnings, 0 errores).

Co-Authored-By: Claude Sonnet 5 <noreply@anthropic.com>
Claude-Session: https://claude.ai/code/session_01T7LXaJdHR17hwkEUJr3uCL
Parts:
- added J19: u.FL, Connector_Coaxial:U.FL_Hirose_U.FL-R-SMT-1_Vertical, symbol Connector:Conn_Coaxial
Connections:
- net GND: now also J19.2 (Ext)
- new net ANT_GNSS: J19.1 (In)
Changed lines of the file:
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@@
+		)
+	)
+	(wire
+		(pts
+			(xy 205.74 179.07) (xy 198.12 179.07)
+		)
+		(stroke
+			(width 0)
+			(type default)
+		)
+	)
+	(wire
+		(pts
+			(xy 210.82 184.15) (xy 210.82 190.5)
+		)
+		(stroke
+			(width 0)
+			(type default)
+		)
+	)
+	(hierarchical_label "ANT_GNSS"
+		(shape passive)
+		(at 198.12 179.07 180)
+		(effects
+			(font
+				(size 1.27 1.27)
+			)
+			(justify right)
+		)
+	)
+	(symbol
+		(lib_id "Connector:Conn_Coaxial")
+		(at 210.82 179.07 0)
+		(unit 1)
+		(exclude_from_sim no)
+		(in_bom yes)
+		(on_board yes)
+		(dnp no)
+		(property "Reference" "J19"
+			(at 210.82 174.07 0)
+			(effects
+				(font
+					(size 1.27 1.27)
+				)
+				(justify left bottom)
+			)
+		)
+		(property "Value" "u.FL"
+			(at 210.82 184.07 0)
+			(effects
+				(font
+					(size 1.27 1.27)
+				)
+				(justify left bottom)
+			)
+		)
+		(property "Footprint" "Connector_Coaxial:U.FL_Hirose_U.FL-R-SMT-1_Vertical"
+			(at 210.82 179.07 0)
+			(effects
+				(font
+					(size 1.27 1.27)
+				)
+				(justify left bottom)
+				(hide yes)
+			)
+		)
+		(property "Datasheet" "https://www.digikey.com/en/products/detail/hirose-electric-co-ltd/U-FL-R-SMT-1-10/2704589"
+			(at 210.82 179.07 0)
+			(effects
+				(font
+					(size 1.27 1.27)
+				)
+				(justify left bottom)
+				(hide yes)
+			)
+		)
+		(property "Description" "Antena GNSS/GPS: pigtail u.FL-u.FL a la toma GNSS de la tarjeta Mini-PCIe (EG25-G / SIM7600). Antena pasiva recomendada (Quectel)."
+			(at 210.82 179.07 0)
+			(effects
+				(font
+					(size 1.27 1.27)
+				)
+				(justify left bottom)
+				(hide yes)
+			)
+		)
+		(property "MPN" "U.FL-R-SMT-1(10)"
+			(at 210.82 179.07 0)
+			(effects
+				(font
+					(size 1.27 1.27)
+				)
+				(justify left bottom)
+				(hide yes)
+			)
+		)
+		(property "MANUFACTURER" "Hirose"
+			(at 210.82 179.07 0)
+			(effects
+				(font
+					(size 1.27 1.27)
+				)
+				(justify left bottom)
+				(hide yes)
+			)
+		)
+		(property "BOM Comments" "Incluye pigtail u.FL-u.FL 100mm a la tarjeta modem; antena GNSS pasiva externa"
+			(at 210.82 179.07 0)
+			(effects
+				(font
+					(size 1.27 1.27)
+				)
+				(justify left bottom)
+				(hide yes)
+			)
+		)
+		(pin "1"
+		)
+		(pin "2"
+		)
+		(instances
+			(project "controlcarreta"
+				(path "/9232987b-e923-413e-abd9-77ced6cc4c47/46e5d0ef-dab9-446e-ac53-867ecc660a13"
+					(reference "J19")
+					(unit 1)
+				)
+			)
+		)
+	)
+	(symbol
+		(lib_id "power:GND")
+		(at 210.82 190.5 0)
+		(unit 1)
+		(exclude_from_sim no)
+		(in_bom yes)
+		(on_board yes)
+		(dnp no)
+		(property "Reference" "#PWR0563"
+			(at 210.82 185.5 0)
+			(effects
+				(font
+					(size 1.27 1.27)
+				)
+				(justify left bottom)
+				(hide yes)
+			)
+		)
+		(property "Value" "GND"
+			(at 210.82 195.5 0)
+			(effects
+				(font
+					(size 1.27 1.27)
+				)
+				(justify left bottom)
+			)
+		)
+		(property "Footprint" ""
+			(at 210.82 190.5 0)
+			(effects
+				(font
+					(size 1.27 1.27)
+				)
+				(justify left bottom)
+				(hide yes)
+			)
+		)
+		(property "Datasheet" "~"
+			(at 210.82 190.5 0)
+			(effects
+				(font
+					(size 1.27 1.27)
+				)
+				(justify left bottom)
+				(hide yes)
+			)
+		)
+		(property "Description" ""
+			(at 210.82 190.5 0)
+			(effects
+				(font
+					(size 1.27 1.27)
+				)
+				(justify left bottom)
+				(hide yes)
+			)
+		)
+		(pin "1"
+		)
+		(instances
+			(project "controlcarreta"
+				(path "/9232987b-e923-413e-abd9-77ced6cc4c47/46e5d0ef-dab9-446e-ac53-867ecc660a13"
+					(reference "#PWR0563")
+					(unit 1)
+				)
+			)
 		)
 	)
