File: modem.kicad_sch (KiCad schematic)
At the start: 10 parts, among them J14 Mini PCIe Socket 52p, J15 nano-SIM, J16 u.FL, J19 u.FL

Commit message: friday changes
Parts:
- C22: DigiKey (none) -> 1276-1003-2-ND; MPN (none) -> CL21B104KBCNNNC; Manufacturer (none) -> Samsung Electro-Mechanics
- D9: DigiKey (none) -> 160-1427-2-ND; MPN (none) -> LTST-C171KRKT; Manufacturer (none) -> Lite-On Inc.
- J14: DigiKey (none) -> 670-2275-2-ND
- J15: DigiKey (none) -> 2223-NSIM-2-CTR-ND
- J16, J19: DigiKey (none) -> H11891TR-ND
- R20, R21: DigiKey (none) -> RMCF1206FT10K0TR-ND; MPN (none) -> RMCF1206FT10K0; Manufacturer (none) -> Stackpole Electronics Inc
- R26: DigiKey (none) -> 311-1.00KFRTR-ND; MPN (none) -> RC1206FR-071KL; Manufacturer (none) -> YAGEO
- R27: DigiKey (none) -> CR1206AJ/-000EASTR-ND; MPN (none) -> CR1206AJ/-000EAS; Manufacturer (none) -> Bourns Inc.

Commit message: schematic updated
Parts:
- added J17: Conn_Coaxial, Connector_Coaxial:SMA_Amphenol_132134-16_Vertical, symbol Connector:Conn_Coaxial
- added J18: SMA GNSS, Connector_Coaxial:SMA_Amphenol_132134-16_Vertical, symbol Connector:Conn_Coaxial
- renumbered C22 to C36, D9 to D4, J16 to J13, J19 to J15, J15 to J16, R20 to R24, R21 to R25, R27 to R26, R26 to R27
Connections:
- net ANT_GNSS: now also J18.1 (In)
- net ANT_MAIN: now also J17.1 (In)
- net GND: now also J17.2 (Ext), J18.2 (Ext)
